File: Omneuro v2/Omneuro v2.kicad_sch (KiCad schematic)
At the start: 90 parts, among them J1 Conn_01x02_Socket, J10 5788800-2, J11 TC2030, J12 Conn_Coaxial, J2 Conn_01x01_Pin, J3 Conn_01x01_Pin, J4 Conn_01x01_Pin, J5 Conn_01x01_Pin, J6 Conn_01x01_Pin, J7 Conn_01x01_Pin, J8 Conn_01x01_Pin, J9 Conn_01x01_Pin, U1 MCP1754T-3302E/OT, U10 TPD4E1B06DRLR, U11 TPD4E1B06DRLR, U12 TPD4E1B06DRLR, U13 ADS1298xPAG, U14 STM32WB55CEU6, U2 LIS3DH, U3 LM2664M6, U4 TLV70025_SOT23-5, U5 SN74LVC1G32DCKR, U6 TPS72325DBV, U7 TPD4E1B06DRLR, U8 TPD4E1B06DRLR, U9 TPD4E1B06DRLR, X1 32.768KHZ

Commit message: update
Parts:
- added D2: LED, symbol Device:LED
- added R13: 220, Resistor_SMD:R_0402_1005Metric, symbol Device:R
- C45: value 0p8 -> 0p3
- J12: footprint (none) -> Connector_Coaxial:U.FL_Hirose_U.FL-R-SMT-1_Vertical
- L1, L2, L3: footprint (none) -> Inductor_SMD:L_0402_1005Metric
- R11, R12: footprint (none) -> Resistor_SMD:R_0402_1005Metric
- U1: value MCP1754T-3302E/OT -> MCP1754T-3302E_OT
Connections:
- net +2V5 is gone; now on net +2.5V: U13.19 (AVDD), U13.21 (AVDD), U13.22 (AVDD), U13.54 (AVDD1), U13.56 (AVDD), U13.59 (AVDD)
- net -2V5 is gone; now on net -2.5V: C22.2, C24.2, C26.2, C28.2, C29.2, C31.2, C33.2, U13.20 (AVSS), U13.23 (AVSS), U13.25 (VREFN), U13.32 (AVSS), U13.53 (AVSS1), U13.57 (AVSS), U13.58 (AVSS)
- net BIAS  is gone; now on net BIAS: J10.10
- net MISO  is gone; now on net MISO: U14.15 (PA6)
- net MOSI  is gone; now on net MOSI: U14.16 (PA7)
- net SLCK is gone; now on net SCLK: U13.40 (SCLK)
- net DRDY: now also U14.45 (PB5)
- net GND: now also R13.1; no longer U13.64 (WCT)
- net INT1: now also U14.14 (PA5)
- net IN_SRB1: now also U13.17 (TESTP_PACE_OUT1)
- net IN_SRB2: now also U13.18 (TESTP_PACE_OUT2)
- net RESET: now also U14.17 (PA8)
- net SRB1: no longer U13.17 (TESTP_PACE_OUT1)
- net SRB2: no longer U13.18 (TESTP_PACE_OUT2)
- net at U14.12 (PA3): now also D2.2 (A)
- new net: D2.1 (K), R13.2
Other:
- note added: "ACC & GYRO"
- note added: "ADC"
- note added: "CONNECTORS & POWER DECOUPLING"
- note added: "MCU"
- note added: "POWER STAGE"
- note added: "TVS CIRCUITRY"
- moved on the sheet: C14, C15, C16, C17, C18, C19, C20, C21, C22, C23, C24, C25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
